Commit message: both finger rviz on

File: finger_tip_rasp_subscribe/urdf/mod_fingertip.urdf.xacro (robot description, xacro)
@@ -3,8 +3,9 @@
        name="left_fingertip_board">
     <xacro:include filename="$(find iai_fingertip_description)/urdf/fingertip_sensor_macro.urdf.xacro" />
-  <xacro:macro name="fingertip_board_xacro" params="prefix parent">
+  <xacro:macro name="fingertip_board_xacro" params="prefix parent base_xyz base_rpy">
     <!-- Joint connecting the parent to our frame_in -->
     <joint name="${prefix}adapter_base_joint" type="fixed">
-      <origin xyz="0 0 0.0" rpy="0 0 0" />
+      <!--<origin xyz="0 0 0.0" rpy="0 0 0" /> -->
+      <origin xyz="${base_xyz}" rpy="${base_rpy}" />
       <parent link="${parent}"/>
       <child link="${prefix}adapter_fingertip_base_frame_in"/>
@@ -67,5 +68,5 @@
    <xacro:vl_sensor suffix="sensor" sens_no ="9" sensor_joint_xyz="0.038 0.065 -0.003" sensor_joint_rpy=" ${-pi/2.0} 0 0 "/>
   </xacro:macro>
-<link name="base_link">
+<link name="fingertip_base_link">
         <visual>
           <geometry>
@@ -74,5 +75,18 @@
           </geometry>
         </visual>
-      </link>
-<xacro:fingertip_board_xacro prefix="left" parent ="base_link" />
+</link>
+    <joint name="base_to_finger" type="fixed">
+      <origin xyz="0 0.5 0" rpy="0 0 0" />
+      <parent link="pbase_link"/>
+      <child link="fingertip_base_link"/>
+    </joint>
+    <!-- Link for the finger sensor-->
+    <link name="pbase_link">
+      <visual>
+        <origin rpy="0 0 0" xyz="0 0 0"/>
+        <material name="White"/>
+      </visual>
+    </link>
+<xacro:fingertip_board_xacro prefix="left" parent ="fingertip_base_link" base_xyz = "-0.5 0.5 0" base_rpy = "0 ${pi/2.0} 0"/>
+<xacro:fingertip_board_xacro prefix="right" parent ="fingertip_base_link" base_xyz = "0.5 0.5 0" base_rpy = "0 ${-pi/2.0} 0"/>
 </robot>
